File: sch/ciot.sch (EAGLE design)
At the start: 38 parts, among them IC1 STM32L051K8U, IC2 TAR5SB30, J1 S2B-PH-SM4-TB, J2 S2B-PH-SM4-TB, U1 MCP73831

Commit message: Update EAGLE files
Parts:
- added C12: 1u, resistor:C-EUC0603K
- C10, C9: value 22p -> 10p
- C5, C6: value 1u -> 0.01u
- R1, R13: value (none) -> 10k
Connections:
- net GND: now also C12.2
- net VDD: now also C12.1
Changed lines of the file:
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@@
 <part name="+3V2" library="supply1" deviceset="+3V3" device=""/>
 <part name="VDD2" library="supply1" deviceset="VDD" device=""/>
-<part name="R1" library="resistor" deviceset="R-EU_" device="R0603"/>
+<part name="R1" library="resistor" deviceset="R-EU_" device="R0603" value="10k"/>
 <part name="SUPPLY3" library="supply2" deviceset="+4.1V" device=""/>
 <part name="IC1" library="micro-stm_v3" deviceset="STM32L051K*U" device="" technology="8"/>
@@
 <part name="VDD5" library="supply1" deviceset="VDD" device=""/>
 <part name="C1" library="resistor" deviceset="C-EU" device="C0603K" value="0.01u"/>
-<part name="C5" library="resistor" deviceset="C-EU" device="C0603K" value="1u"/>
-<part name="C6" library="resistor" deviceset="C-EU" device="C0603K" value="1u"/>
+<part name="C5" library="resistor" deviceset="C-EU" device="C0603K" value="0.01u"/>
+<part name="C6" library="resistor" deviceset="C-EU" device="C0603K" value="0.01u"/>
 <part name="GND10" library="supply1" deviceset="GND" device=""/>
 <part name="VDD6" library="supply1" deviceset="VDD" device=""/>
@@
 <part name="GND14" library="supply1" deviceset="GND" device=""/>
 <part name="GND16" library="supply1" deviceset="GND" device=""/>
-<part name="R13" library="resistor" deviceset="R-EU_" device="R0603"/>
+<part name="R13" library="resistor" deviceset="R-EU_" device="R0603" value="10k"/>
 <part name="U$3" library="crystal" deviceset="FC-255" device=""/>
-<part name="C9" library="resistor" deviceset="C-EU" device="C0603K" value="22p"/>
-<part name="C10" library="resistor" deviceset="C-EU" device="C0603K" value="22p"/>
+<part name="C9" library="resistor" deviceset="C-EU" device="C0603K" value="10p"/>
+<part name="C10" library="resistor" deviceset="C-EU" device="C0603K" value="10p"/>
 <part name="GND17" library="supply1" deviceset="GND" device=""/>
 <part name="GND24" library="supply1" deviceset="GND" device=""/>
@@
 <part name="GND22" library="supply1" deviceset="GND" device=""/>
 <part name="VDD13" library="supply1" deviceset="VDD" device=""/>
+<part name="C12" library="resistor" deviceset="C-EU" device="C0603K" value="1u"/>
+<part name="VDD14" library="supply1" deviceset="VDD" device=""/>
+<part name="GND26" library="supply1" deviceset="GND" device=""/>
 </parts>
 <sheets>
@@
 <instance part="VDD12" gate="G$1" x="157.48" y="111.76"/>
 <instance part="VDD13" gate="G$1" x="48.26" y="111.76"/>
+<instance part="C12" gate="G$1" x="243.84" y="157.48"/>
+<instance part="VDD14" gate="G$1" x="243.84" y="165.1"/>
+<instance part="GND26" gate="1" x="243.84" y="147.32"/>
 </instances>
 <busses>
@@
 <wire x1="48.26" y1="93.98" x2="48.26" y2="109.22" width="0.1524" layer="91"/>
 <pinref part="VDD13" gate="G$1" pin="VDD"/>
+</segment>
+<segment>
+<pinref part="C12" gate="G$1" pin="1"/>
+<pinref part="VDD14" gate="G$1" pin="VDD"/>
+<wire x1="243.84" y1="160.02" x2="243.84" y2="162.56" width="0.1524" layer="91"/>
 </segment>
 </net>
@@
 <wire x1="157.48" y1="101.6" x2="157.48" y2="99.06" width="0.1524" layer="91"/>
 </segment>
+<segment>
+<pinref part="C12" gate="G$1" pin="2"/>
+<pinref part="GND26" gate="1" pin="GND"/>
+<wire x1="243.84" y1="149.86" x2="243.84" y2="152.4" width="0.1524" layer="91"/>
+</segment>
 </net>
